File: cbm-d9096.kicad_pcb (KiCad board)
At the start: 2 copper layers, 90.2 x 68.6 mm, 32 parts, among them J1 IEEE488 Header, J2 SD CARD, J3 WP/CD Jumper, J4 LED, J5 RESET, J6 Barrel_Jack, J7 Alt PWR, U1 ATmega1284-P, U2 75160, U3 75161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

Commit message: RN1 Description fix
RN1 was described as 6x10K, changed to the correct 5*6K
Parts:
- RN1: value 6x10K -> 5x10K
